File: current_measurer.sch (KiCad schematic (older format))
At the start: 15 parts, among them J1 Eurorack Power Input, J2 Eurorack Power Output, J3 Back_Conn_2, J4 Front_Conn_2, J5 Back_Conn_3, J6 Front_Conn_3, J7 Back_Conn_1, J8 Front_Conn_1, SW1 SW_Push, U1 L7805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

Commit message: Add extra pin for VIN
Parts:
- added J9: VIN, Connector_Wire:SolderWire-0.5sqmm_1x01_D0.9mm_OD2.1mm, symbol Connector_Generic:Conn_01x01
Connections:
- net at A1.30 (VIN): now also J9.1 (Pin_1)
- no-connect marks 32 -> 31
Changed lines of the file:
@@
 	1900 2600 1900 2450
 NoConn ~ 1800 2600
-NoConn ~ 1600 2600
 NoConn ~ 2200 3400
 NoConn ~ 2200 3100
@@
 U 1 1 6163ADCC
 P 1700 3600
-F 0 "A1" H 1300 4800 50  0000 C CNN
-F 1 "Arduino_Nano_v3.x" H 1300 4900 50  0000 C CNN
+F 0 "A1" H 1050 4500 50  0000 C CNN
+F 1 "Arduino_Nano_v3.x" H 900 4600 50  0000 C CNN
 F 2 "jwm_kicad_footprints_misc:Arduino_Nano_WithMFHeadersAnd3DModel" H 1700 3600 50  0001 C CIN
 F 3 "http://www.mouser.com/pdfdocs/Gravitech_Arduino_Nano3_0.pdf" H 1700 3600 50  0001 C CNN
@@
 Text Notes 6550 5750 0    50   ~ 0
  PCB2\n(Panel)
+$Comp
+L Connector_Generic:Conn_01x01 J9
+U 1 1 6190B91D
+P 1600 2250
+F 0 "J9" V 1800 2300 50  0000 R CNN
+F 1 "VIN" V 1700 2300 50  0000 R CNN
+F 2 "Connector_Wire:SolderWire-0.5sqmm_1x01_D0.9mm_OD2.1mm" H 1600 2250 50  0001 C CNN
+F 3 "~" H 1600 2250 50  0001 C CNN
+	1    1600 2250
+	0    -1   -1   0
+$EndComp
+Wire Wire Line
+	1600 2600 1600 2450
 $EndSCHEMATC
